Commit message: Parse the model file using xacro and set tf_prefix.

File: src/grex/models/robots/waffle.model.xacro (robot description, xacro)
@@ -1,6 +1,8 @@
 <?xml version="1.0" ?>
-<sdf version="1.5">
+<sdf version="1.5" xmlns:xacro="http://ros.org/wiki/xacro">
+  <xacro:arg name="tf_prefix" default=""/>
+  <xacro:property name="tf_prefix" value="$(arg tf_prefix)"/>
   <model name="turtlebot3_waffle">
-  <pose>0.0 0.0 0.0 0.0 0.0 0.0</pose>
+    <pose>0.0 0.0 0.0 0.0 0.0 0.0</pose>
     <link name="base_footprint"/>
     <link name="base_link">
@@ -151,5 +153,5 @@
           </ros>
           <output_type>sensor_msgs/LaserScan</output_type>
-          <frame_name>base_scan</frame_name>
+          <frame_name>${tf_prefix}base_scan</frame_name>
         </plugin>
       </sensor>
@@ -464,6 +466,6 @@
       <publish_wheel_tf>false</publish_wheel_tf>
       <odometry_topic>odom</odometry_topic>
-      <odometry_frame>odom</odometry_frame>
-      <robot_base_frame>base_footprint</robot_base_frame>
+      <odometry_frame>${tf_prefix}odom</odometry_frame>
+      <robot_base_frame>${tf_prefix}base_footprint</robot_base_frame>
     </plugin>
     <plugin name="turtlebot3_joint_state" filename="libgazebo_ros_joint_state_publisher.so">
